Commit message: Add OmniHand MuJoCo visualization

File: wuji_retargeting/omnihand_description/urdf/omnihand_left.urdf (robot description, URDF)
Before this commit: robot omnihand, 24 links, 23 joints
Links:
- link L_index_abad: geometry visual mesh filename=../meshes/finger_abad.STL
- link L_index_dip: geometry collision cylinder length=0.034 radius=0.007; visual mesh filename=../meshes/finger_dip.STL
- link L_index_pip: geometry collision cylinder length=0.044 radius=0.01; visual mesh filename=../meshes/finger_pip.STL
- link L_middle_abad: geometry visual mesh filename=../meshes/finger_abad.STL
- link L_middle_dip: geometry collision cylinder length=0.034 radius=0.007; visual mesh filename=../meshes/finger_dip.STL
- link L_middle_pip: geometry collision cylinder length=0.044 radius=0.01; visual mesh filename=../meshes/finger_pip.STL
- link L_palm: geometry collision box size=0.04 0.082 0.085; collision cylinder length=0.0145 radius=0.028
- link L_pinky_abad: geometry visual mesh filename=../meshes/finger_abad.STL
- link L_pinky_dip: geometry collision cylinder length=0.034 radius=0.007; visual mesh filename=../meshes/finger_dip.STL
- link L_pinky_pip: geometry collision cylinder length=0.044 radius=0.01; visual mesh filename=../meshes/finger_pip.STL
- link L_ring_abad: geometry visual mesh filename=../meshes/finger_abad.STL
- link L_ring_dip: geometry collision cylinder length=0.034 radius=0.007; visual mesh filename=../meshes/finger_dip.STL
- link L_ring_pip: geometry collision cylinder length=0.044 radius=0.01; visual mesh filename=../meshes/finger_pip.STL
- link L_thumb_abad: geometry visual mesh filename=../meshes/thumb_abad.STL
- link L_thumb_dip: geometry collision cylinder length=0.023 radius=0.011; visual mesh filename=../meshes/thumb_dip.STL
- link L_thumb_mcp: geometry collision box size=0.029 0.042 0.0325; visual mesh filename=../meshes/thumb_mcp.STL
- link L_thumb_pip: geometry collision box size=0.019 0.035 0.0225; visual mesh filename=../meshes/thumb_pip.STL
- link L_thumb_roll: geometry visual mesh filename=../meshes/l_thumb_roll.STL

File: wuji_retargeting/omnihand_description/urdf/omnihand_right.urdf (robot description, URDF)
Before this commit: robot omnihand, 24 links, 23 joints
Links:
- link R_index_abad: geometry visual mesh filename=../meshes/finger_abad.STL
- link R_index_dip: geometry collision cylinder length=0.034 radius=0.007; visual mesh filename=../meshes/finger_dip.STL
- link R_index_pip: geometry collision cylinder length=0.044 radius=0.01; visual mesh filename=../meshes/finger_pip.STL
- link R_middle_abad: geometry visual mesh filename=../meshes/finger_abad.STL
- link R_middle_dip: geometry collision cylinder length=0.034 radius=0.007; visual mesh filename=../meshes/finger_dip.STL
- link R_middle_pip: geometry collision cylinder length=0.044 radius=0.01; visual mesh filename=../meshes/finger_pip.STL
- link R_palm: geometry collision box size=0.04 0.082 0.085; collision cylinder length=0.0145 radius=0.028
- link R_pinky_abad: geometry visual mesh filename=../meshes/finger_abad.STL
- link R_pinky_dip: geometry collision cylinder length=0.034 radius=0.007; visual mesh filename=../meshes/finger_dip.STL
- link R_pinky_pip: geometry collision cylinder length=0.044 radius=0.01; visual mesh filename=../meshes/finger_pip.STL
- link R_ring_abad: geometry visual mesh filename=../meshes/finger_abad.STL
- link R_ring_dip: geometry collision cylinder length=0.034 radius=0.007; visual mesh filename=../meshes/finger_dip.STL
- link R_ring_pip: geometry collision cylinder length=0.044 radius=0.01; visual mesh filename=../meshes/finger_pip.STL
- link R_thumb_abad: geometry visual mesh filename=../meshes/thumb_abad.STL
- link R_thumb_dip: geometry collision cylinder length=0.023 radius=0.011; visual mesh filename=../meshes/thumb_dip.STL
- link R_thumb_mcp: geometry collision box size=0.029 0.042 0.0325; visual mesh filename=../meshes/thumb_mcp.STL
- link R_thumb_pip: geometry collision box size=0.019 0.035 0.0225; visual mesh filename=../meshes/thumb_pip.STL
- link R_thumb_roll: geometry visual mesh filename=../meshes/r_thumb_roll.STL
